Commit message: fetch_camera addition
added fetch camera so it can be integrated

File: fetch_robotdata/robots/fetch_camera.urdf (robot description, URDF)
Before this commit: robot fetch, 7 links, 6 joints
Links:
- link base_link: geometry collision mesh filename=fetch_robotdata/meshes/base_link_collision.STL
- link head_pan_link: geometry collision mesh filename=fetch_robotdata/meshes/head_pan_link_collision.STL; visual mesh filename=fetch_robotdata/meshes/head_pan_link.dae
- link head_tilt_link: geometry collision mesh filename=fetch_robotdata/meshes/head_tilt_link_collision.STL; visual mesh filename=fetch_robotdata/meshes/head_tilt_link.dae
- link torso_lift_link: geometry collision mesh filename=fetch_robotdata/meshes/torso_lift_link_collision.STL
