Commit message: updated .urdf so robot works
the no limits resulted in robot not working in ikine IT NOW WORKS THANK GOD

File: fetch_robotdata/robots/fetch.urdf (robot description, URDF)
Before this commit: robot fetch, 19 links, 18 joints
Joints:
- joint base_joint1: limit lower=-999999 upper=999999 effort=87 velocity=4.0 -> lower=-10 upper=10 effort=87 velocity=4.0
- joint base_joint2: limit lower=-999999 upper=999999 effort=87 velocity=4.0 -> lower=-10 upper=10 effort=87 velocity=4.0
- joint forearm_roll_joint: limit effort=29.35 velocity=1.571 -> lower=-1.5707 upper=1.5707 effort=29.35 velocity=1.571
- joint upperarm_roll_joint: limit effort=76.94 velocity=1.571 -> lower=-1.5707 upper=1.5707 effort=76.94 velocity=1.571
- joint wrist_roll_joint: limit effort=7.36 velocity=2.268 -> lower=-1.5707 upper=1.5707 effort=7.36 velocity=2.268

Commit message: fixed urdf so it should work on everyones compq
doesnt look at the robotics package but the folder inside the repo so should work for everyone now

File: fetch_robotdata/robots/fetch.urdf (robot description, URDF)
Before this commit: robot fetch, 19 links, 18 joints
Links:
- link base_link: geometry collision mesh filename=fetch_robotdata/meshes/base_link_collision.STL; visual mesh filename=fetch_robotdata/meshes/base_link.dae
- link bellows_link: geometry collision mesh filename=fetch_robotdata/meshes/bellows_link_collision.STL; visual mesh filename=fetch_robotdata/meshes/bellows_link.STL
- link bellows_link2: geometry collision mesh filename=fetch_robotdata/meshes/bellows_link_collision.STL; visual mesh filename=fetch_robotdata/meshes/bellows_link.STL
- link elbow_flex_link: geometry collision mesh filename=fetch_robotdata/meshes/elbow_flex_link_collision.STL; visual mesh filename=fetch_robotdata/meshes/elbow_flex_link.dae
- link estop_link: geometry collision mesh filename=fetch_robotdata/meshes/estop_link.STL; visual mesh filename=fetch_robotdata/meshes/estop_link.dae
- link forearm_roll_link: geometry collision mesh filename=fetch_robotdata/meshes/forearm_roll_link_collision.STL; visual mesh filename=fetch_robotdata/meshes/forearm_roll_link.dae
- link gripper_link: geometry collision mesh filename=fetch_robotdata/meshes/gripper_link.STL; visual mesh filename=fetch_robotdata/meshes/gripper_link.dae
- link l_gripper_finger_link: geometry collision mesh filename=fetch_robotdata/meshes/l_gripper_finger_link.STL; visual mesh filename=fetch_robotdata/meshes/l_gripper_finger_link.STL
- link laser_link: geometry collision mesh filename=fetch_robotdata/meshes/laser_link.STL; visual mesh filename=fetch_robotdata/meshes/laser_link.STL
- link r_gripper_finger_link: geometry collision mesh filename=fetch_robotdata/meshes/r_gripper_finger_link.STL; visual mesh filename=fetch_robotdata/meshes/r_gripper_finger_link.STL
- link shoulder_lift_link: geometry collision mesh filename=fetch_robotdata/meshes/shoulder_lift_link_collision.STL; visual mesh filename=fetch_robotdata/meshes/shoulder_lift_link.dae
- link shoulder_pan_link: geometry collision mesh filename=fetch_robotdata/meshes/shoulder_pan_link_collision.STL; visual mesh filename=fetch_robotdata/meshes/shoulder_pan_link.dae
- link torso_fixed_link: geometry collision mesh filename=fetch_robotdata/meshes/torso_fixed_link.STL; visual mesh filename=fetch_robotdata/meshes/torso_fixed_link.dae
- link torso_lift_link: geometry collision mesh filename=fetch_robotdata/meshes/torso_lift_link_collision.STL; visual mesh filename=fetch_robotdata/meshes/torso_lift_link.dae
- link upperarm_roll_link: geometry collision mesh filename=fetch_robotdata/meshes/upperarm_roll_link_collision.STL; visual mesh filename=fetch_robotdata/meshes/upperarm_roll_link.dae
- link wrist_flex_link: geometry collision mesh filename=fetch_robotdata/meshes/wrist_flex_link_collision.STL; visual mesh filename=fetch_robotdata/meshes/wrist_flex_link.dae
- link wrist_roll_link: geometry collision mesh filename=fetch_robotdata/meshes/wrist_roll_link_collision.STL; visual mesh filename=fetch_robotdata/meshes/wrist_roll_link.dae

Commit message: its broken for some reason but now its in the krustykrab

File: fetch_robotdata/robots/fetch.urdf (robot description, URDF)
Before this commit: robot fetch, 19 links, 18 joints
Joints:
- joint base_joint2: limit lower=-10 upper=10 effort=87 velocity=4.0 -> lower=-20 upper=20 effort=87 velocity=4.0
